File: v1.0/Hardware/SynchronousRectifier.kicad_sch (KiCad schematic)
At the start: 15 parts, among them J1 MAINS_IN, U1 4N39, U2 4N39

Commit message: v1.1&v1.2 PCB addition.
#####v1.1#####
+Change of MCU; STM32F334C8T6 instead of STM32F103C8T6.
+Filtering 3rd order components of the square wave.
+Use  4 capacitors.
+Adapted to generic transformer(primary 6.4mH, secondary 14.4mH)
+Faster IGBT.

########v1.2#######
+Measures only PZT current and voltage.
+Differential inputs.
+Analog circuitry is capable of measuring four quadrant voltage, current and complex impedance.
+Half bridge configuration.
+Gate resistance of the IGBT's lowered.
+Only USART based touch panel can be connected; not conventional LCD.
Other:
- note added: "Notes: Replace R1&R2 with 10k resistors to ease triggering since PC13-PC14 pins can only sink 3miliamps."
Changed lines of the file:
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@@
 (kicad_sch (version 20200506) (host eeschema "5.99.0-unknown-1f9723c~101~ubuntu18.04.1")
   (page "A4")
+  (junction (at 151.765 95.25))
+  (junction (at 157.48 120.65))
+  (junction (at 122.555 95.25))
+  (junction (at 151.765 120.65))
   (junction (at 140.335 120.65))
-  (junction (at 151.765 120.65))
-  (junction (at 122.555 95.25))
+  (junction (at 99.06 111.76))
+  (junction (at 160.655 120.65))
+  (junction (at 106.68 106.68))
+  (junction (at 146.05 95.25))
+  (junction (at 160.655 95.25))
+  (junction (at 132.08 109.22))
+  (junction (at 99.06 106.68))
+  (junction (at 132.08 120.65))
+  (junction (at 146.05 120.65))
+  (junction (at 110.49 109.22))
+  (junction (at 122.555 106.68))
   (junction (at 132.08 95.25))
-  (junction (at 110.49 109.22))
-  (junction (at 146.05 120.65))
-  (junction (at 157.48 120.65))
-  (junction (at 106.68 106.68))
-  (junction (at 122.555 106.68))
   (junction (at 130.175 109.22))
+  (junction (at 157.48 95.25))
+  (junction (at 140.335 95.25))
   (junction (at 101.6 109.22))
-  (junction (at 132.08 120.65))
-  (junction (at 157.48 95.25))
-  (junction (at 99.06 111.76))
-  (junction (at 146.05 95.25))
-  (junction (at 132.08 109.22))
-  (junction (at 160.655 95.25))
-  (junction (at 99.06 106.68))
-  (junction (at 151.765 95.25))
-  (junction (at 160.655 120.65))
-  (junction (at 140.335 95.25))
   (wire (pts (xy 97.155 106.68) (xy 99.06 106.68)))
   (wire (pts (xy 97.155 109.22) (xy 101.6 109.22)))
@@
   (wire (pts (xy 162.56 82.55) (xy 163.83 82.55)))
   (wire (pts (xy 162.56 99.695) (xy 162.56 100.33)))
+  (polyline (pts (xy 104.14 27.94) (xy 104.14 52.705)))
+  (polyline (pts (xy 104.14 27.94) (xy 171.45 27.94)))
+  (polyline (pts (xy 104.14 52.705) (xy 171.45 52.705)))
+  (polyline (pts (xy 171.45 52.705) (xy 171.45 27.94)))
+  (text "Notes:\nReplace R1&R2 with 10k resistors to ease triggering since \nPC13-PC14 pins can only sink 3miliamps."
+    (at 106.68 36.195 0)
+    (effects (font (size 1.27 1.27)) (justify left bottom))
+  )
   (hierarchical_label "T0_TRIGGER" (shape input) (at 163.83 71.755 0)
     (effects (font (size 1.27 1.27)) (justify left))
