File: v1.1/Hardware/IsensAfe.kicad_sch (KiCad schematic)
At the start: 37 parts, among them Q15 MMBT3904, Q16 MMBT3904, U13 L78L05_SOT89, U3 MCP6024, U4 ACPL-7900, U5 TL431LP

Commit message: v1.1&v1.2 PCB addition.
#####v1.1#####
+Change of MCU; STM32F334C8T6 instead of STM32F103C8T6.
+Filtering 3rd order components of the square wave.
+Use  4 capacitors.
+Adapted to generic transformer(primary 6.4mH, secondary 14.4mH)
+Faster IGBT.

########v1.2#######
+Measures only PZT current and voltage.
+Differential inputs.
+Analog circuitry is capable of measuring four quadrant voltage, current and complex impedance.
+Half bridge configuration.
+Gate resistance of the IGBT's lowered.
+Only USART based touch panel can be connected; not conventional LCD.
Parts:
- C10, C11, C22, C24, C5, C8, C9: footprint Capacitor_SMD:C_0805_2012Metric_Pad1.15x1.40mm_HandSolder -> Capacitor_SMD:C_0805_2012Metric
- C4: value 10n -> 100n; footprint Resistor_SMD:R_0805_2012Metric_Pad1.15x1.40mm_HandSolder -> Resistor_SMD:R_0805_2012Metric; Link https://ozdisan.com/passive-components/capacitors/smt-smd-and-mlcc-capacitors/CL21B103KCANNNC -> https://ozdisan.com/passive-components/capacitors/smt-smd-and-mlcc-capacitors/CL21B104KBFWPNE; Price 0.05749TL -> 0.10509TL
- C6, C7: value 150p -> 330p; footprint Capacitor_SMD:C_0805_2012Metric_Pad1.15x1.40mm_HandSolder -> Capacitor_SMD:C_0805_2012Metric; Link https://ozdisan.com/passive-components/capacitors/smt-smd-and-mlcc-capacitors/CL21C181JBANNNC -> https://ozdisan.com/passive-components/capacitors/smt-smd-and-mlcc-capacitors/CL21C331JCANNNC; Price 0.09416TL -> 0.08531TL
- R10, R11, R16, R17, R18, R20, R21, R22, R23, R33, R34, R5, R52, R6, R7, R8, R9: footprint Resistor_SMD:R_0805_2012Metric_Pad1.15x1.40mm_HandSolder -> Resistor_SMD:R_0805_2012Metric
- U5: symbol Reference_Voltage:TL431LP -> Reference_Voltage:TL431DBZ; Link https://ozdisan.com/integrated-circuits-ics/power-management-ics/voltage-reference-ics/TL431NSG-AE2-R -> https://ozdisan.com/integrated-circuits-ics/power-management-ics/voltage-reference-ics/TL431AIDBZR; Price 0.46403TL -> 0.88437TL
Connections:
- net GND: now also U5.3 (A); no longer U5.2 (A)
- net at R20.1, R22.1, U5.1 (K): now also U5.2 (REF); no longer U5.3 (K)
