File: v1.1/Hardware/PowerSources.kicad_sch (KiCad schematic)
At the start: 63 parts, among them Q10 BC556, Q11 BC546, Q12 BC556, Q13 BC546, Q14 BC556, Q5 BC546, Q6 BC556, Q7 BC546, Q8 BC556, Q9 BC546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

Commit message: v1.1&v1.2 PCB addition.
#####v1.1#####
+Change of MCU; STM32F334C8T6 instead of STM32F103C8T6.
+Filtering 3rd order components of the square wave.
+Use  4 capacitors.
+Adapted to generic transformer(primary 6.4mH, secondary 14.4mH)
+Faster IGBT.

########v1.2#######
+Measures only PZT current and voltage.
+Differential inputs.
+Analog circuitry is capable of measuring four quadrant voltage, current and complex impedance.
+Half bridge configuration.
+Gate resistance of the IGBT's lowered.
+Only USART based touch panel can be connected; not conventional LCD.
Parts:
- removed C13: 10uF, Capacitor_Tantalum_SMD:CP_EIA-6032-15_Kemet-U_Pad2.25x2.35mm_HandSolder, symbol Device:CP_Small
- removed U6: AMS1117-5.0, Package_TO_SOT_SMD:SOT-223-3_TabPin2, symbol Regulator_Linear:AMS1117-5.0
- added C74: 100n, Capacitor_SMD:C_0805_2012Metric, symbol Device:C_Small
- added C75: 10uF, Capacitor_Tantalum_SMD:CP_EIA-6032-15_Kemet-U, symbol Device:CP_Small
- added C76: 1000u 35v, Capacitor_THT:CP_Radial_D12.5mm_P5.00mm, symbol Device:CP
- added L1: EMIFilter_LL_2314, oe_inductor:EPCOS_B82721A, symbol oe_choke:EMIFilter_LL_2314
- added U6: L7805, Package_TO_SOT_SMD:TO-252-2, symbol Regulator_Linear:L7805
- C12, C14: footprint Capacitor_SMD:C_0805_2012Metric_Pad1.15x1.40mm_HandSolder -> Capacitor_SMD:C_0805_2012Metric
- C40: value 10uF -> 1uF 35v; footprint Capacitor_Tantalum_SMD:CP_EIA-6032-15_Kemet-U_Pad2.25x2.35mm_HandSolder -> Capacitor_SMD:C_1206_3216Metric; Link https://ozdisan.com/passive-components/capacitors/tantalum-capacitors/T491C106K025AT -> https://ozdisan.com/passive-components/capacitors/tantalum-capacitors/T491A105K035AT; Price 1.59678TL -> 0.66495TL
- C67: footprint Capacitor_Tantalum_SMD:CP_EIA-6032-15_Kemet-U_Pad2.25x2.35mm_HandSolder -> Capacitor_Tantalum_SMD:CP_EIA-6032-15_Kemet-U
Connections:
- net +5V: now also C74.2, C75.1, U6.3 (OUT)
- net GND: now also C74.1, C75.2, U6.2 (GND)
- net GND1: now also L1.4
- net VCC: now also U6.1 (IN)
- net VEE: now also L1.2
- new net GND2: C76.2, L1.3
- new net Vdrive: C76.1, L1.1
Other:
- moved on the sheet: C40
