File: v1.1/Hardware/WaveUltrasonics.kicad_pcb (KiCad board)
At the start: 2 copper layers, 300 x 155 mm, 217 parts, among them J1 MAINS_IN, J2 Conn_02x08_Counter_Clockwise, J3 TRANSDUCER, J4 FAN, J5 Conn_01x04, J6 Conn_01x04, Q1 IXXH80N65B4H1, Q10 BC556, Q11 BC546, Q12 BC556, Q13 BC546, Q14 BC556, Q15 MMBT3904, Q16 MMBT3904, Q17 MMBT3904, Q2 IXXH80N65B4H1, Q3 IXXH80N65B4H1, Q4 IXXH80N65B4H1, Q5 BC546, Q6 BC556, Q7 BC546, Q8 BC556, Q9 BC546, T1 Transformer_1P_1S, T2 Transformer_1P_2S, T3 Transformer_1P_2S, T4 Transformer_1P_2S, U1 4N39, U10 HCPL-3120, U11 HCPL-3120, U12 OPA228, U13 L78L05_SOT89, U14 TLV1117-33, U15 STM32F103CBTx, U16 ADuM1201AR, U2 4N39, U3 MCP6024, U4 ACPL-7900, U5 TL431LP, U6 AMS1117-5.0, U7 TLV73333PDBV, U8 HCPL-3120, U9 HCPL-3120, Y1 8MHz

Commit message: v1.1&v1.2 PCB addition.
#####v1.1#####
+Change of MCU; STM32F334C8T6 instead of STM32F103C8T6.
+Filtering 3rd order components of the square wave.
+Use  4 capacitors.
+Adapted to generic transformer(primary 6.4mH, secondary 14.4mH)
+Faster IGBT.

########v1.2#######
+Measures only PZT current and voltage.
+Differential inputs.
+Analog circuitry is capable of measuring four quadrant voltage, current and complex impedance.
+Half bridge configuration.
+Gate resistance of the IGBT's lowered.
+Only USART based touch panel can be connected; not conventional LCD.
Parts:
- removed D30: RED LED, LED_SMD:LED_0805_2012Metric_Pad1.15x1.40mm_HandSolder
- removed L2: 4.11mH, oe_inductor:Toroid_21mm_38mm
- removed R35, R36: 120R, Resistor_THT:R_Axial_DIN0207_L6.3mm_D2.5mm_P10.16mm_Horizontal
- removed R54, R55, R56, R57: 1k, Resistor_SMD:R_0805_2012Metric_Pad1.15x1.40mm_HandSolder
- removed R60: 220R, Resistor_SMD:R_0805_2012Metric_Pad1.15x1.40mm_HandSolder
- removed T1: Transformer_1P_1S, oe_transformer:Toroid_2x2_26mm_55mm
- added C68: 100n, Capacitor_SMD:C_0805_2012Metric, F.Cu at (132.8, 202.4)
- added C69: 470u 400v, oe_capacitor:CP_Radial_D35.0mm_P10.00mm_SnapIn, F.Cu at (269.2, 115.7)
- added C70: 100n, Capacitor_SMD:C_0805_2012Metric, F.Cu at (120.8, 162.8)
- added C71: 100n, Capacitor_SMD:C_0805_2012Metric, F.Cu at (121.4, 158.6)
- added C72: 10n, Capacitor_THT:C_Rect_L18.0mm_W5.0mm_P15.00mm_FKS3_FKP3, F.Cu at (285.9, 180.8)
- added C73: 2.2n 400VAC, Capacitor_THT:C_Rect_L13.0mm_W4.0mm_P10.00mm_FKS3_FKP3_MKS4, F.Cu at (295.4, 160.5)
- added C74: 100n, Capacitor_SMD:C_0805_2012Metric, F.Cu at (135.6, 148.1)
- added C75: 10uF, Capacitor_Tantalum_SMD:CP_EIA-6032-15_Kemet-U, F.Cu at (125.2, 138.3)
- added C76: 1000u 35v, Capacitor_THT:CP_Radial_D12.5mm_P5.00mm, F.Cu at (73.2, 146.6)
- added C77: 100n, Capacitor_SMD:C_0805_2012Metric, F.Cu at (137.9, 184.0)
- added J10: DG25C-B-04P-13-00AH, oe_connector:DG25C-B-04P-13-00AH, F.Cu at (312.5, 151.6)
- added J7: DS1069-02MVW6X, Connector_JST:JST_EH_B2B-EH-A_1x02_P2.50mm_Vertical, F.Cu at (127.1, 208.8)
- added J8: DS1069-04MVW6X, Connector_JST:JST_EH_B4B-EH-A_1x04_P2.50mm_Vertical, F.Cu at (148.1, 208.8)
- added J9: DG25C-B-04P-13-00AH, oe_connector:DG25C-B-04P-13-00AH, F.Cu at (312.5, 187.2)
- added Q18: MMBT3904, Package_TO_SOT_SMD:SOT-23, F.Cu at (139.2, 202.8)
- added Q19: MMBT3904, Package_TO_SOT_SMD:SOT-23, F.Cu at (143.0, 202.8)
- added Q20: MMBT3904, Package_TO_SOT_SMD:SOT-23, F.Cu at (146.8, 202.8)
- added Q21: BC817, Package_TO_SOT_SMD:SOT-23, F.Cu at (163.3, 122.4)
- added Q22: BC817, Package_TO_SOT_SMD:SOT-23, F.Cu at (163.3, 134.5)
- added Q23: BC817, Package_TO_SOT_SMD:SOT-23, F.Cu at (160.8, 169.4)
- added Q24: BC817, Package_TO_SOT_SMD:SOT-23, F.Cu at (160.8, 148.5)
- added Q25: BC817, Package_TO_SOT_SMD:SOT-23, F.Cu at (160.8, 185.9)
- added Q26: BC817, Package_TO_SOT_SMD:SOT-23, F.Cu at (160.8, 201.8)
- added Q27: BC817, Package_TO_SOT_SMD:SOT-23, F.Cu at (141.9, 157.1)
- added R61: 120R, Resistor_SMD:R_0805_2012Metric, F.Cu at (100.5, 202.4)
- added R62: 4.7k, Resistor_SMD:R_0805_2012Metric, F.Cu at (159.5, 121.8)
- added R63: 2.2k, Resistor_SMD:R_0805_2012Metric, F.Cu at (159.5, 124.3)
- added R64: 4.7k, Resistor_SMD:R_0805_2012Metric, F.Cu at (159.5, 133.9)
- added R65: 2.2k, Resistor_SMD:R_0805_2012Metric, F.Cu at (159.5, 136.4)
- added R67: 120R, Resistor_SMD:R_0805_2012Metric, F.Cu at (157.0, 168.1)
- added R68: 120R, Resistor_SMD:R_0805_2012Metric, F.Cu at (157.0, 147.8)
- added R69: 8.2k, Resistor_SMD:R_0805_2012Metric, F.Cu at (160.8, 172.6)
- added R70: 8.2k, Resistor_SMD:R_0805_2012Metric, F.Cu at (160.8, 151.6)
- added R71: 82R, Resistor_SMD:R_0805_2012Metric, F.Cu at (160.8, 166.2)
- added R72: 82R, Resistor_SMD:R_0805_2012Metric, F.Cu at (160.8, 145.3)
- added R73: 22k 7W, Resistor_THT:R_Axial_DIN0922_L20.0mm_D9.0mm_P30.48mm_Horizontal, F.Cu at (291.6, 97.0)
- added R74: 22k 7W, Resistor_THT:R_Axial_DIN0922_L20.0mm_D9.0mm_P30.48mm_Horizontal, F.Cu at (291.6, 92.6)
- added R75: 4.7k 5W, Resistor_THT:R_Axial_Power_L25.0mm_W9.0mm_P30.48mm, F.Cu at (279.5, 160.5)
- added R76: 4.7k 5W, Resistor_THT:R_Axial_Power_L25.0mm_W9.0mm_P30.48mm, F.Cu at (279.5, 182.1)
- added R77: 4.7k 5W, Resistor_THT:R_Axial_Power_L25.0mm_W9.0mm_P30.48mm, F.Cu at (279.5, 171.3)
- added R78: 82R, Resistor_SMD:R_0805_2012Metric, F.Cu at (160.8, 182.8)
- added R79: 82R, Resistor_SMD:R_0805_2012Metric, F.Cu at (160.8, 198.6)
- added R80: 8.2k, Resistor_SMD:R_0805_2012Metric, F.Cu at (160.8, 189.1)
- added R81: 120R, Resistor_SMD:R_0805_2012Metric, F.Cu at (157.0, 184.7)
- added R82: 8.2k, Resistor_SMD:R_0805_2012Metric, F.Cu at (160.8, 205.0)
- added R83: 120R, Resistor_SMD:R_0805_2012Metric, F.Cu at (157.0, 200.5)
- added R84: 120R, Resistor_SMD:R_0805_2012Metric, F.Cu at (137.9, 182.1)
- added R85: 2.2k, Resistor_SMD:R_0805_2012Metric, F.Cu at (141.9, 160.1)
- added TP13: TestPoint_2Pole, Connector_PinHeader_2.54mm:PinHeader_1x02_P2.54mm_Vertical, F.Cu at (99.2, 137.0)
- added TP14: TestPoint_2Pole, Connector_PinHeader_2.54mm:PinHeader_1x02_P2.54mm_Vertical, F.Cu at (107.4, 137.0)
- added U17: STM32F334C8Tx, Package_QFP:LQFP-48_7x7mm_P0.5mm, F.Cu at (110.6, 177.0)
- C10, C11, C12, C14, C22, C24, C49, C5, C50, C59, C60, C61, C62, C63, C64, C65, C66, C8, C9: footprint Capacitor_SMD:C_0805_2012Metric_Pad1.15x1.40mm_HandSolder -> Capacitor_SMD:C_0805_2012Metric
- C13: value 10uF -> 1u; footprint Capacitor_Tantalum_SMD:CP_EIA-6032-15_Kemet-U_Pad2.25x2.35mm_HandSolder -> Capacitor_SMD:C_0805_2012Metric
- C15, C39: footprint Capacitor_SMD:C_0603_1608Metric_Pad1.05x0.95mm_HandSolder -> Capacitor_SMD:C_0603_1608Metric
- C26: value 1.5n 400VAC -> 100n; footprint Capacitor_THT:C_Rect_L18.0mm_W5.0mm_P15.00mm_FKS3_FKP3 -> Capacitor_SMD:C_0805_2012Metric
- C27, C28, C30, C32, C34: value 22n 400VAC -> 6.8n 400VAC
- C29, C31, C33, C35: value 220n 310VAC -> 10n; footprint Capacitor_THT:C_Rect_L18.0mm_W8.0mm_P15.00mm_FKS3_FKP3 -> Capacitor_THT:C_Rect_L18.0mm_W5.0mm_P15.00mm_FKS3_FKP3
- C4: value 10n -> 100n; footprint Resistor_SMD:R_0805_2012Metric_Pad1.15x1.40mm_HandSolder -> Resistor_SMD:R_0805_2012Metric
- C40: value 10uF -> 1uF 35v; footprint Capacitor_Tantalum_SMD:CP_EIA-6032-15_Kemet-U_Pad2.25x2.35mm_HandSolder -> Capacitor_SMD:C_1206_3216Metric
- C48: footprint Capacitor_THT:C_Rect_L7.2mm_W2.5mm_P5.00mm_FKS2_FKP2_MKS2_MKP2 -> Capacitor_SMD:C_0805_2012Metric
- C6, C7: value 150p -> 330p; footprint Capacitor_SMD:C_0805_2012Metric_Pad1.15x1.40mm_HandSolder -> Capacitor_SMD:C_0805_2012Metric
- C67: footprint Capacitor_Tantalum_SMD:CP_EIA-6032-15_Kemet-U_Pad2.25x2.35mm_HandSolder -> Capacitor_Tantalum_SMD:CP_EIA-6032-15_Kemet-U
- D1, D3: value CLA30E1200HB -> CLA50E1200HB
- D2, D4: value DSEP30-06A -> DSEI60-06A
- D29: value BLUE LED -> SMAJ6R0CA-HT; footprint LED_SMD:LED_0805_2012Metric_Pad1.15x1.40mm_HandSolder -> oe_diode:DO214AC_SMA
- J2: value Conn_02x08_Counter_Clockwise -> L-KLS1-207-2-12-S; footprint Connector_PinHeader_2.54mm:PinHeader_2x08_P2.54mm_Vertical -> Connector_PinHeader_2.54mm:PinHeader_2x06_P2.54mm_Vertical
- J3: value TRANSDUCER -> Screw_Terminal_01x03
- J4: value FAN -> DS1069-02MVW6X; footprint oe_connector:DG128-5.0-02P-14-00AH -> Connector_JST:JST_EH_B2B-EH-A_1x02_P2.50mm_Vertical
- J6: value Conn_01x04 -> DS1069-04MVW6X; footprint Connector_PinHeader_2.54mm:PinHeader_1x04_P2.54mm_Vertical -> Connector_JST:JST_EH_B4B-EH-A_1x04_P2.50mm_Vertical
- L1: value 264.4u 20A -> EMIFilter_LL_2314; footprint oe_inductor:Toroid_21mm_38mm -> oe_inductor:EPCOS_B82721A
- R1, R2: value 1k -> 1.5k; footprint Resistor_THT:R_Axial_DIN0204_L3.6mm_D1.6mm_P5.08mm_Horizontal -> Resistor_THT:R_Axial_DIN0204_L3.6mm_D1.6mm_P7.62mm_Horizontal
- R10, R11, R16, R17, R18, R20, R21, R22, R23, R33, R34, R47, R48, R5, R51, R52, R53, R59, R6, R7, R8, R9: footprint Resistor_SMD:R_0805_2012Metric_Pad1.15x1.40mm_HandSolder -> Resistor_SMD:R_0805_2012Metric
- R12, R13: value 120R -> 10k; footprint Resistor_THT:R_Axial_DIN0207_L6.3mm_D2.5mm_P10.16mm_Horizontal -> Resistor_SMD:R_0805_2012Metric
- R14, R15, R31, R32: value 4.7R -> 10R
- R26: value 0.33R 5W -> 10k; footprint Resistor_THT:R_Axial_Power_L25.0mm_W9.0mm_P30.48mm -> Resistor_SMD:R_0805_2012Metric
- R27: value 3.3k 7W -> 10k; footprint Resistor_THT:R_Axial_Power_L25.0mm_W9.0mm_P30.48mm -> Resistor_SMD:R_0805_2012Metric
- R28: value 3.3k 7W -> 2.2k; footprint Resistor_THT:R_Axial_Power_L25.0mm_W9.0mm_P30.48mm -> Resistor_SMD:R_0805_2012Metric
- R29, R30: value 0.33R 5W -> 120R; footprint Resistor_THT:R_Axial_Power_L25.0mm_W9.0mm_P30.48mm -> Resistor_SMD:R_0805_2012Metric
- R3, R4: value 120R -> 51R 1/2Watt; footprint Resistor_THT:R_Axial_DIN0207_L6.3mm_D2.5mm_P10.16mm_Horizontal -> Resistor_SMD:R_1210_3225Metric
- R49, R50: value 270k -> 1M; footprint Resistor_SMD:R_0805_2012Metric_Pad1.15x1.40mm_HandSolder -> Resistor_SMD:R_0805_2012Metric
- R58: value 2.2k -> 10k; footprint Resistor_SMD:R_0805_2012Metric_Pad1.15x1.40mm_HandSolder -> Resistor_SMD:R_0805_2012Metric
- U15: value STM32F103CBTx -> 4N25; footprint Package_QFP:LQFP-48_7x7mm_P0.5mm -> Package_DIP:DIP-6_W7.62mm
- U16: value ADuM1201AR -> ADM2483xRW; footprint Package_SO:SOIC-8_3.9x4.9mm_P1.27mm -> Package_SO:SOIC-16W_7.5x10.3mm_P1.27mm
- U6: value AMS1117-5.0 -> L7805; footprint Package_TO_SOT_SMD:SOT-223-3_TabPin2 -> Package_TO_SOT_SMD:TO-252-2
- moved L1 273.2 mm to (72.5, 130.7), turned to 0 degrees
- moved R27 234.5 mm to (120.1, 194.2)
- moved C26 229.7 mm to (124.0, 192.3), turned to 180 degrees
- moved R28 218.9 mm to (127.8, 192.3), turned to 180 degrees
- moved R30 128.9 mm to (120.1, 201.2), turned to -90 degrees
- moved R29 117.7 mm to (132.8, 205.0)
- moved R26 101.7 mm to (147.4, 199.0), turned to -90 degrees
- moved TP6 92.4 mm to (266.2, 146.6), turned to 0 degrees
- moved G*** 71.7 mm to (141.7, 120.9)
- moved C13 66.7 mm to (66.2, 151.0), turned to 180 degrees
- moved C2 60.2 mm to (269.4, 78.3)
- moved TP11 56.8 mm to (308.7, 128.8)
- moved R12 55.0 mm to (139.8, 199.0), turned to -90 degrees
- moved R59 54.1 mm to (153.2, 208.8), turned to 0 degrees
- moved J1 49.8 mm to (312.5, 81.2), turned to -90 degrees
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Connections:
- net /GATE2_GND renamed /RSENS+
- C13 pad 1: +5V -> GND2
- C13 pad 2: GND -> Vdrive
- C26 pad 1: Net-(C25-Pad1) -> VDD
- C26 pad 2: Net-(C25-Pad2) -> GND
- C29 pad 1: Net-(C29-Pad1) -> /GATE3_GND
- C31 pad 1: Net-(C29-Pad1) -> /GATE3_GND
- C33 pad 1: Net-(C29-Pad1) -> /GATE3_GND
- C35 pad 1: Net-(C29-Pad1) -> /GATE3_GND
- C48 pad 1: GND1 -> GND2
- C48 pad 2: VEE -> Vdrive
- D29 pad 1: GND -> Net-(D29-Pad1)
- J2 pad 10: /Mcu/LCD_BSENS -> /Mcu/LCD_EN
- J2 pad 11: /Mcu/LCD_D6 -> /Mcu/LCD_RS
- J2 pad 12: /Mcu/LCD_EN -> /Mcu/LCD_R~W
- J2 pad 3: /Mcu/A1 -> /Mcu/LCD_D7
- J2 pad 5: /Mcu/B9 -> /Mcu/LCD_D6
- J2 pad 6: /Mcu/B15 -> Net-(J2-Pad6)
- J2 pad 7: /Mcu/B8 -> /Mcu/LCD_D5
- J2 pad 8: /Mcu/LCD_BKLIT -> /Mcu/LCD_BSENS
- J2 pad 9: /Mcu/LCD_D7 -> /Mcu/LCD_D4
- J3 pad 2: Net-(J3-Pad2) -> Net-(J10-Pad3)
- J4 pad 1: VEE -> Vdrive
- J4 pad 2: GND1 -> GND2
- L1 pad 1: Net-(C29-Pad2) -> Vdrive
- L1 pad 2: Net-(C27-Pad1) -> VEE
- R12 pad 1: Net-(R12-Pad1) -> /LED_RED
- R12 pad 2: /HBRIDGE_A_HSIDE -> Net-(Q18-Pad1)
- R13 pad 1: Net-(R13-Pad1) -> /LED_GREEN
- R13 pad 2: /HBRIDGE_A_LSIDE -> Net-(Q19-Pad1)
- R26 pad 1: /GATE3_GND -> /LED_BLUE
- R26 pad 2: Net-(C29-Pad1) -> Net-(Q20-Pad1)
- R27 pad 1: Net-(C25-Pad2) -> GND
- R27 pad 2: Net-(J3-Pad2) -> Net-(R27-Pad2)
- R28 pad 1: Net-(C25-Pad2) -> /TRIGOUT
- R28 pad 2: Net-(J3-Pad2) -> VDD
- R29 pad 1: /GATE3_GND -> Net-(D29-Pad1)
- R29 pad 2: Net-(C29-Pad1) -> +5V
- R3 pad 1: /THRISTOR0_DRV -> Net-(R3-Pad1)
- R3 pad 2: Net-(R3-Pad2) -> +5V
- R30 pad 1: /GATE3_GND -> GND
- R30 pad 2: Net-(C29-Pad1) -> Net-(D29-Pad2)
- R4 pad 1: /THRISTOR1_DRV -> Net-(R4-Pad1)
- R4 pad 2: Net-(R4-Pad2) -> +5V
- R58 pad 1: GND -> Net-(R58-Pad1)
- R58 pad 2: Net-(R58-Pad2) -> GND
- R59 pad 1: /LED_BLUE -> Net-(J8-Pad1)
- R59 pad 2: Net-(D29-Pad2) -> +5V
- TP11 pad 1: Net-(J3-Pad2) -> Net-(J10-Pad3)
- U1 pad 1: Net-(R3-Pad2) -> Net-(R3-Pad1)
- U1 pad 2: GND -> Net-(Q21-Pad3)
- U15 pad 1: VDD -> Net-(D29-Pad1)
- U15 pad 2: (no net) -> Net-(D29-Pad2)
- U15 pad 4: (no net) -> GND
- U15 pad 5: Net-(C15-Pad2) -> /TRIGOUT
- U15 pad 6: Net-(C39-Pad2) -> Net-(R27-Pad2)
- U16 pad 2: /SELF_IN -> GND
- U16 pad 3: /USART_TX -> /RS485_RX
- U16 pad 4: GND -> /RS485_DE~RE
- U16 pad 5: Net-(C66-Pad1) -> /RS485_DE~RE
- U16 pad 6: Net-(J6-Pad3) -> /RS485_TX
- U16 pad 7: Net-(J6-Pad2) -> (no net)
- U16 pad 8: Net-(C66-Pad2) -> GND
- U2 pad 1: Net-(R4-Pad2) -> Net-(R4-Pad1)
- U2 pad 2: GND -> Net-(Q22-Pad3)
- U5 pad 2: GND -> Net-(R20-Pad1)
- U5 pad 3: Net-(R20-Pad1) -> GND
- U6 pad 1: GND -> VCC
- U6 pad 2: +5V -> GND
- U6 pad 3: VCC -> +5V
- U8 pad 2: Net-(R12-Pad1) -> Net-(Q24-Pad3)
- U9 pad 2: Net-(R13-Pad1) -> Net-(Q23-Pad3)
Routing:
- net Net-(J10-Pad3): track 0.00 -> 200.7 mm, vias 0 -> 1
- net /~HBRIDGE_A_HSIDE: track 0.00 -> 68.2 mm, vias 0 -> 4
- net +5V: track 96.0 -> 30.3 mm, vias 7 -> 1
- net /~HBRIDGE_B_LSIDE: track 0.00 -> 62.1 mm, vias 0 -> 4
- net /Mcu/B15: track 57.0 -> 0.00 mm, vias 3 -> 0
- net GND2: track 0.00 -> 55.9 mm, vias 0 -> 1
- net /Mcu/A1: track 54.0 -> 0.00 mm, vias 6 -> 0
- net /HBRIDGE_B_LSIDE: track 53.4 -> 0.00 mm, vias 2 -> 0
- net /HBRIDGE_A_HSIDE: track 52.9 -> 0.00 mm, vias 2 -> 0
- net Net-(C6-Pad2): track 6.86 -> 58.5 mm, vias 0 -> 11
- net /~HBRIDGE_A_LSIDE: track 0.00 -> 47.7 mm, vias 0 -> 4
- net Earth_Protective: track 85.6 -> 38.3 mm
- net /LED_GREEN: track 0.00 -> 47.0 mm, vias 0 -> 6
- net +VDC: track 212.0 -> 165.3 mm, vias 3 -> 4
- net /Mcu/LCD_BKLIGHT: track 0.00 -> 46.6 mm, vias 0 -> 4
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- added copper zone on F.Cu, net +5V
- added copper zone on F.Cu, net /RSENS+
- added copper zone on B.Cu, net Net-(C25-Pad1)
- added copper zone on B.Cu, net Net-(J10-Pad3)
- removed copper zone on F.Cu, net Net-(C25-Pad1)
- removed copper zone on F.Cu, net Net-(C25-Pad2)
- removed copper zone on F.Cu, net Net-(C29-Pad1)
- removed copper zone on F.Cu, net Net-(J3-Pad2)
Other:
- board size 300 x 155 mm -> 262 x 155 mm
- net class Gnd: trace_width 0.6 -> 0.5; via_drill 0.9 -> 0.8
- net class Low Power: trace_width 0.6 -> 0.5; via_dia 1.25 -> 1.2
- net class Mid Power: trace_width 0.85 -> 0.75; via_dia 1.4 -> 1.8; via_drill 1 -> 1.2
- board text added: "A"
- board text added: "B"
- board text added: "BKLIT"
- board text added: "BSENS"
- board text added: "D4"
- board text added: "D5"
- board text added: "D6"
- board text added: "D7"
- board text added: "INDCOMP_A"
- board text added: "INDCOMP_B"
- board text added: "INDFILT_A"
- board text added: "INDFILT_B"
- board text added: "INVIPRO"
- board text added: "IOVER"
- board text added: "LDA"
- board text added: "LDB"
- board text added: "LDG"
- board text added: "LDR"
- board text added: "PHASE+"
- board text added: "TRGA"
- board text added: "TRGB"
- board text added: "TRPRI_A"
- board text added: "TRPRI_B"
- board text added: "TRSEC_A"
- board text added: "TRSEC_B"
- board text added: "ZCROSS"
- board text removed: "A1"
- board text removed: "B0"
- board text removed: "B15"
- board text removed: "B8"
- board text removed: "B9"
- board text removed: "BL"
- board text removed: "DAT4"
- board text removed: "DAT5"
- board text removed: "DAT6"
- board text removed: "DAT7"
- board text removed: "INV_CURR_PROTECT"
- board text removed: "OVERCURRENT"
- board text removed: "RX"
- board text removed: "TX"

Commit message: Start of rs485 communication interface development.
Other:
- net class Default removed
- net class Gnd removed
- net class High power removed
- net class Low Power removed
- net class Mid Power removed
