File: v1.2/Hardware/PowerSources.kicad_sch (KiCad schematic)
At the start: 45 parts, among them Q10 BC556, Q5 BC546, Q6 BC556, Q7 BC546, Q8 BC556, Q9 BC546, T2 Transformer_1P_2S, T3 Transformer_1P_2S, U14 TLV1117-33, U6 L7805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

Commit message: Redesign.
+Cli interface.
+Modularity improvement(complex number and pid modules created)
+Range change.
+Core-Lattice seperated. 
+Improvement of the control function
Changed lines of the file:
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@@
-(kicad_sch (version 20200618) (host eeschema "5.99.0-unknown-f3f1740~101~ubuntu18.04.1")
+(kicad_sch (version 20200828) (generator eeschema)
   (page 7 8)
   (paper "A4")
-  (junction (at 57.785 101.6) (diameter 0) (color 0 0 0 0))
-  (junction (at 66.675 109.855) (diameter 0) (color 0 0 0 0))
-  (junction (at 72.39 40.005) (diameter 0) (color 0 0 0 0))
-  (junction (at 74.295 32.385) (diameter 0) (color 0 0 0 0))
-  (junction (at 75.565 101.6) (diameter 0) (color 0 0 0 0))
-  (junction (at 77.47 32.385) (diameter 0) (color 0 0 0 0))
-  (junction (at 86.995 63.5) (diameter 0) (color 0 0 0 0))
-  (junction (at 88.9 32.385) (diameter 0) (color 0 0 0 0))
-  (junction (at 88.9 40.005) (diameter 0) (color 0 0 0 0))
-  (junction (at 88.9 48.26) (diameter 0) (color 0 0 0 0))
-  (junction (at 92.71 63.5) (diameter 0) (color 0 0 0 0))
-  (junction (at 92.71 83.82) (diameter 0) (color 0 0 0 0))
-  (junction (at 93.98 32.385) (diameter 0) (color 0 0 0 0))
-  (junction (at 94.615 126.365) (diameter 0) (color 0 0 0 0))
-  (junction (at 95.25 102.235) (diameter 0) (color 0 0 0 0))
-  (junction (at 95.885 126.365) (diameter 0) (color 0 0 0 0))
-  (junction (at 97.155 32.385) (diameter 0) (color 0 0 0 0))
-  (junction (at 97.155 40.005) (diameter 0) (color 0 0 0 0))
-  (junction (at 103.505 30.48) (diameter 0) (color 0 0 0 0))
-  (junction (at 103.505 37.465) (diameter 0) (color 0 0 0 0))
-  (junction (at 103.505 42.545) (diameter 0) (color 0 0 0 0))
-  (junction (at 103.505 49.53) (diameter 0) (color 0 0 0 0))
-  (junction (at 113.03 102.235) (diameter 0) (color 0 0 0 0))
-  (junction (at 114.3 126.365) (diameter 0) (color 0 0 0 0))
-  (junction (at 114.935 63.5) (diameter 0) (color 0 0 0 0))
-  (junction (at 114.935 83.82) (diameter 0) (color 0 0 0 0))
-  (junction (at 193.04 79.375) (diameter 0) (color 0 0 0 0))
-  (junction (at 193.04 99.695) (diameter 0) (color 0 0 0 0))
-  (junction (at 203.2 63.5) (diameter 0) (color 0 0 0 0))
-  (junction (at 203.2 73.025) (diameter 0) (color 0 0 0 0))
-  (junction (at 203.2 82.55) (diameter 0) (color 0 0 0 0))
-  (junction (at 203.2 96.52) (diameter 0) (color 0 0 0 0))
-  (junction (at 203.2 106.045) (diameter 0) (color 0 0 0 0))
-  (junction (at 203.2 115.57) (diameter 0) (color 0 0 0 0))
-  (junction (at 207.01 73.025) (diameter 0) (color 0 0 0 0))
-  (junction (at 207.01 106.045) (diameter 0) (color 0 0 0 0))
-  (junction (at 213.36 63.5) (diameter 0) (color 0 0 0 0))
-  (junction (at 213.36 70.485) (diameter 0) (color 0 0 0 0))
-  (junction (at 213.36 75.565) (diameter 0) (color 0 0 0 0))
-  (junction (at 213.36 82.55) (diameter 0) (color 0 0 0 0))
-  (junction (at 213.36 96.52) (diameter 0) (color 0 0 0 0))
-  (junction (at 213.36 103.505) (diameter 0) (color 0 0 0 0))
-  (junction (at 213.36 108.585) (diameter 0) (color 0 0 0 0))
-  (junction (at 213.36 115.57) (diameter 0) (color 0 0 0 0))
-  (junction (at 234.315 63.5) (diameter 0) (color 0 0 0 0))
-  (junction (at 234.315 73.025) (diameter 0) (color 0 0 0 0))
-  (junction (at 234.315 82.55) (diameter 0) (color 0 0 0 0))
-  (junction (at 234.315 96.52) (diameter 0) (color 0 0 0 0))
-  (junction (at 234.315 106.045) (diameter 0) (color 0 0 0 0))
-  (junction (at 234.315 115.57) (diameter 0) (color 0 0 0 0))
+  (junction (at 57.785 101.6) (diameter 0.3048) (color 0 0 0 0))
+  (junction (at 66.675 109.855) (diameter 0.3048) (color 0 0 0 0))
+  (junction (at 72.39 40.005) (diameter 0.3048) (color 0 0 0 0))
+  (junction (at 74.295 32.385) (diameter 0.3048) (color 0 0 0 0))
+  (junction (at 75.565 101.6) (diameter 0.3048) (color 0 0 0 0))
+  (junction (at 77.47 32.385) (diameter 0.3048) (color 0 0 0 0))
+  (junction (at 86.995 63.5) (diameter 0.3048) (color 0 0 0 0))
+  (junction (at 88.9 32.385) (diameter 0.3048) (color 0 0 0 0))
+  (junction (at 88.9 40.005) (diameter 0.3048) (color 0 0 0 0))
+  (junction (at 88.9 48.26) (diameter 0.3048) (color 0 0 0 0))
+  (junction (at 92.71 63.5) (diameter 0.3048) (color 0 0 0 0))
+  (junction (at 92.71 83.82) (diameter 0.3048) (color 0 0 0 0))
+  (junction (at 93.98 32.385) (diameter 0.3048) (color 0 0 0 0))
+  (junction (at 94.615 126.365) (diameter 0.3048) (color 0 0 0 0))
+  (junction (at 95.25 102.235) (diameter 0.3048) (color 0 0 0 0))
+  (junction (at 95.885 126.365) (diameter 0.3048) (color 0 0 0 0))
+  (junction (at 97.155 32.385) (diameter 0.3048) (color 0 0 0 0))
+  (junction (at 97.155 40.005) (diameter 0.3048) (color 0 0 0 0))
+  (junction (at 103.505 30.48) (diameter 0.3048) (color 0 0 0 0))
+  (junction (at 103.505 37.465) (diameter 0.3048) (color 0 0 0 0))
+  (junction (at 103.505 42.545) (diameter 0.3048) (color 0 0 0 0))
+  (junction (at 103.505 49.53) (diameter 0.3048) (color 0 0 0 0))
+  (junction (at 113.03 102.235) (diameter 0.3048) (color 0 0 0 0))
+  (junction (at 114.3 126.365) (diameter 0.3048) (color 0 0 0 0))
+  (junction (at 114.935 63.5) (diameter 0.3048) (color 0 0 0 0))
+  (junction (at 114.935 83.82) (diameter 0.3048) (color 0 0 0 0))
+  (junction (at 193.04 79.375) (diameter 0.3048) (color 0 0 0 0))
+  (junction (at 193.04 99.695) (diameter 0.3048) (color 0 0 0 0))
+  (junction (at 203.2 63.5) (diameter 0.3048) (color 0 0 0 0))
+  (junction (at 203.2 73.025) (diameter 0.3048) (color 0 0 0 0))
+  (junction (at 203.2 82.55) (diameter 0.3048) (color 0 0 0 0))
+  (junction (at 203.2 96.52) (diameter 0.3048) (color 0 0 0 0))
+  (junction (at 203.2 106.045) (diameter 0.3048) (color 0 0 0 0))
+  (junction (at 203.2 115.57) (diameter 0.3048) (color 0 0 0 0))
+  (junction (at 207.01 73.025) (diameter 0.3048) (color 0 0 0 0))
+  (junction (at 207.01 106.045) (diameter 0.3048) (color 0 0 0 0))
+  (junction (at 213.36 63.5) (diameter 0.3048) (color 0 0 0 0))
+  (junction (at 213.36 70.485) (diameter 0.3048) (color 0 0 0 0))
+  (junction (at 213.36 75.565) (diameter 0.3048) (color 0 0 0 0))
+  (junction (at 213.36 82.55) (diameter 0.3048) (color 0 0 0 0))
+  (junction (at 213.36 96.52) (diameter 0.3048) (color 0 0 0 0))
+  (junction (at 213.36 103.505) (diameter 0.3048) (color 0 0 0 0))
+  (junction (at 213.36 108.585) (diameter 0.3048) (color 0 0 0 0))
+  (junction (at 213.36 115.57) (diameter 0.3048) (color 0 0 0 0))
+  (junction (at 234.315 63.5) (diameter 0.3048) (color 0 0 0 0))
+  (junction (at 234.315 73.025) (diameter 0.3048) (color 0 0 0 0))
+  (junction (at 234.315 82.55) (diameter 0.3048) (color 0 0 0 0))
+  (junction (at 234.315 96.52) (diameter 0.3048) (color 0 0 0 0))
+  (junction (at 234.315 106.045) (diameter 0.3048) (color 0 0 0 0))
+  (junction (at 234.315 115.57) (diameter 0.3048) (color 0 0 0 0))
   (wire (pts (xy 38.1 35.56) (xy 38.1 37.465))
     (stroke (width 0) (type solid) (color 0 0 0 0))
