File: v1.3/Hardware/PowerInput.kicad_sch (KiCad schematic)
At the start: 12 parts, among them J1 DG25C-B-03P-13-00AH

Commit message: v1.3 Schematic, footprints and BOM updated.
Parts:
- removed D?: GBJ5010-BP, symbol Device:D_Bridge_+AA-
- added D1, D2, D3, D4: DSEI60-06A, Package_TO_SOT_THT:TO-247-2_Vertical, symbol Device:D_Small
- D5: renamed from D?; footprint (none) -> Diode_SMD:D_SMA
- R1: renamed from R?; footprint (none) -> Resistor_THT:R_Axial_Power_L25.0mm_W9.0mm_P30.48mm
- U1: renamed from U?; footprint (none) -> oe_relay:ALZN5B12W
- gave numbers to parts that had none: 2
Connections:
- net -VDC: now also D2.2 (A), D4.2 (A)
- net LINE: now also D1.2 (A), D2.1 (K)
- net NEUT: now also D3.2 (A), D4.1 (K)
- net at R1.1, U1.4 (COM), U1.5: now also D1.1 (K), D3.1 (K)
- net +12V renamed VCC
