File: v1.3/Hardware/HalfBridge.kicad_sch (KiCad schematic)
At the start: 49 parts, among them J10 DG25C-B-04P-13-00AH, J3 DG25C-B-03P-13-00AH, J4 DG25C-B-03P-13-00AH, Q1 IXGH48N60C3D1, Q2 IXGH48N60C3D1, Q23 MMBT3904, Q24 MMBT3904, U8 HCPL-3120, U9 HCPL-3120

Commit message: v1.3 Layout added & schematic update.
Parts:
- removed C20, C37: 820n 400VDC, Capacitor_THT:C_Rect_L24.0mm_W10.1mm_P22.50mm_MKT, symbol Device:C_Small
Changed lines of the file:
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@@
   (junction (at 114.935 82.55) (diameter 0.3048) (color 0 0 0 0))
   (junction (at 114.935 103.505) (diameter 0.3048) (color 0 0 0 0))
-  (junction (at 119.38 71.12) (diameter 0.3048) (color 0 0 0 0))
   (junction (at 119.38 78.105) (diameter 0.3048) (color 0 0 0 0))
   (junction (at 123.19 71.12) (diameter 0.3048) (color 0 0 0 0))
-  (junction (at 123.19 78.105) (diameter 0.3048) (color 0 0 0 0))
-  (junction (at 127 71.12) (diameter 0.3048) (color 0 0 0 0))
   (junction (at 132.08 71.12) (diameter 0.3048) (color 0 0 0 0))
   (junction (at 132.08 88.265) (diameter 0.3048) (color 0 0 0 0))
@@
     (stroke (width 0) (type solid) (color 0 0 0 0))
   )
-  (wire (pts (xy 115.57 71.12) (xy 119.38 71.12))
-    (stroke (width 0) (type solid) (color 0 0 0 0))
-  )
-  (wire (pts (xy 115.57 72.39) (xy 115.57 71.12))
-    (stroke (width 0) (type solid) (color 0 0 0 0))
-  )
-  (wire (pts (xy 115.57 77.47) (xy 115.57 78.105))
-    (stroke (width 0) (type solid) (color 0 0 0 0))
-  )
-  (wire (pts (xy 115.57 78.105) (xy 119.38 78.105))
-    (stroke (width 0) (type solid) (color 0 0 0 0))
-  )
   (wire (pts (xy 116.84 88.265) (xy 114.935 88.265))
     (stroke (width 0) (type solid) (color 0 0 0 0))
@@
     (stroke (width 0) (type solid) (color 0 0 0 0))
   )
-  (wire (pts (xy 123.19 71.12) (xy 127 71.12))
+  (wire (pts (xy 123.19 71.12) (xy 132.08 71.12))
     (stroke (width 0) (type solid) (color 0 0 0 0))
   )
   (wire (pts (xy 123.19 77.47) (xy 123.19 78.105))
-    (stroke (width 0) (type solid) (color 0 0 0 0))
-  )
-  (wire (pts (xy 123.19 78.105) (xy 127 78.105))
-    (stroke (width 0) (type solid) (color 0 0 0 0))
-  )
-  (wire (pts (xy 127 71.12) (xy 127 72.39))
-    (stroke (width 0) (type solid) (color 0 0 0 0))
-  )
-  (wire (pts (xy 127 71.12) (xy 132.08 71.12))
-    (stroke (width 0) (type solid) (color 0 0 0 0))
-  )
-  (wire (pts (xy 127 77.47) (xy 127 78.105))
     (stroke (width 0) (type solid) (color 0 0 0 0))
   )
@@
     )
   )
-  (symbol (lib_name "Device:C_Small_19") (lib_id "Device:C_Small") (at 115.57 74.93 180) (unit 1)
-    (in_bom yes) (on_board yes)
-    (property "Reference" "C20" (id 0) (at 116.205 69.85 90))
-    (property "Value" "820n 400VDC" (id 1) (at 114.3 69.85 90))
-    (property "Footprint" "Capacitor_THT:C_Rect_L24.0mm_W10.1mm_P22.50mm_MKT" (id 2) (at 115.57 74.93 0)
-      (effects (font (size 1.27 1.27)) hide)
-    )
-    (property "Datasheet" "~" (id 3) (at 115.57 74.93 0)
-      (effects (font (size 1.27 1.27)) hide)
-    )
-    (property "Link" "https://ozdisan.com/passive-components/capacitors/film-capacitors/TMCF03-824K400VP22-5B" (id 4) (at 115.57 74.93 90)
-      (effects (font (size 1.27 1.27)) hide)
-    )
-    (property "Price" "0.11041 USD" (id 5) (at 115.57 74.93 90)
-      (effects (font (size 1.27 1.27)) hide)
-    )
-  )
   (symbol (lib_name "Device:C_Small_17") (lib_id "Device:C_Small") (at 119.38 74.93 180) (unit 1)
     (in_bom yes) (on_board yes)
@@
       (effects (font (size 1.27 1.27)) hide)
     )
-  )
-  (symbol (lib_name "Device:C_Small_6") (lib_id "Device:C_Small") (at 127 74.93 180) (unit 1)
-    (in_bom yes) (on_board yes)
-    (property "Reference" "C37" (id 0) (at 127.635 69.85 90))
-    (property "Value" "820n 400VDC" (id 1) (at 125.73 69.85 90))
-    (property "Footprint" "Capacitor_THT:C_Rect_L24.0mm_W10.1mm_P22.50mm_MKT" (id 2) (at 127 74.93 0)
-      (effects (font (size 1.27 1.27)) hide)
-    )
-    (property "Datasheet" "~" (id 3) (at 127 74.93 0)
-      (effects (font (size 1.27 1.27)) hide)
-    )
-    (property "Link" "https://ozdisan.com/passive-components/capacitors/film-capacitors/TMCF03-824K400VP22-5B" (id 4) (at 127 74.93 90)
-      (effects (font (size 1.27 1.27)) hide)
-    )
-    (property "Price" "0.11041 USD" (id 5) (at 127 74.93 90)
-      (effects (font (size 1.27 1.27)) hide)
-    )
