File: v1.3/Hardware/Mcu.kicad_sch (KiCad schematic)
At the start: 15 parts, among them J2 L-KLS1-207-2-08-S, J5 Conn_01x04, U17 STM32F334C8Tx, Y1 8MHz

Commit message: Serial interface development. Manual added. Untested.
Changed lines of the file:
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@@
-(kicad_sch (version 20200714) (host eeschema "5.99.0-unknown-4b7c88309~102~ubuntu18.04.1")
-  (page 5 7)
+(kicad_sch (version 20201015) (generator eeschema)
+  (page 1 7)
   (paper "A4")
   (junction (at 109.855 66.04) (diameter 0.3048) (color 0 0 0 0))
@@
   (junction (at 211.455 71.755) (diameter 0.3048) (color 0 0 0 0))
   (junction (at 227.965 71.755) (diameter 0.3048) (color 0 0 0 0))
+  (no_connect (at 167.005 100.33))
   (no_connect (at 133.985 85.09))
+  (no_connect (at 133.985 105.41))
+  (no_connect (at 133.985 74.93))
+  (no_connect (at 167.005 120.65))
+  (no_connect (at 167.005 107.95))
+  (no_connect (at 167.005 110.49))
+  (no_connect (at 167.005 97.79))
+  (no_connect (at 133.985 72.39))
+  (no_connect (at 167.005 113.03))
+  (no_connect (at 133.985 82.55))
   (no_connect (at 133.985 77.47))
-  (no_connect (at 133.985 74.93))
-  (no_connect (at 167.005 107.95))
-  (no_connect (at 167.005 113.03))
   (no_connect (at 133.985 120.65))
-  (no_connect (at 133.985 82.55))
-  (no_connect (at 167.005 97.79))
-  (no_connect (at 133.985 105.41))
-  (no_connect (at 167.005 100.33))
-  (no_connect (at 133.985 72.39))
-  (no_connect (at 167.005 120.65))
-  (no_connect (at 167.005 110.49))
   (wire (pts (xy 71.12 38.1) (xy 72.39 38.1))
     (stroke (width 0) (type solid) (color 0 0 0 0))
@@
     (in_bom yes) (on_board yes)
     (property "Reference" "U17" (id 0) (at 150.495 127.8954 0))
-    (property "Value" "STM32F334C8Tx" (id 1) (at 150.495 130.1941 0))
+    (property "Value" "STM32F334C8Tx" (id 1) (at 173.355 69.2341 0))
     (property "Footprint" "Package_QFP:LQFP-48_7x7mm_P0.5mm" (id 2) (at 136.525 123.19 0)
       (effects (font (size 1.27 1.27)) (justify right) hide)

Commit message: v1.3 Schematic, footprints and BOM updated.
Parts:
- removed C70, C71: 100n, Capacitor_SMD:C_0805_2012Metric, symbol Device:C_Small
- removed J2: L-KLS1-207-2-08-S, Connector_PinHeader_2.54mm:PinHeader_2x04_P2.54mm_Vertical, symbol Connector_Generic:Conn_02x04_Odd_Even
- removed J5: Conn_01x04, Connector_PinHeader_2.54mm:PinHeader_1x04_P2.54mm_Vertical, symbol Connector_Generic:Conn_01x04
- added C13, C32, C33, C34: 100n, Capacitor_SMD:C_0805_2012Metric, symbol Device:C_Small
- added J2: Conn_01x05, Connector_PinHeader_2.54mm:PinHeader_1x05_P2.54mm_Vertical, symbol Connector_Generic:Conn_01x05
- added J5: Conn_01x08, Connector_PinHeader_2.54mm:PinHeader_1x08_P2.54mm_Vertical, symbol Connector_Generic:Conn_01x08
Connections:
- net HMI_SELF_RX is gone; now on net MISC1: U17.43 (PB7)
- net HMI_SELF_TX is gone; now on net MISC0: U17.42 (PB6)
- net +5V: now also C32.1, J5.2 (Pin_2)
- net GND: now also C13.1, C32.2, C33.2, C34.2, J2.5 (Pin_5), J5.6 (Pin_6), J5.7 (Pin_7), J5.8 (Pin_8)
- net MISC0: now also J5.5 (Pin_5); no longer U17.39 (PB3)
- net MISC1: now also J5.4 (Pin_4); no longer U17.40 (PB4)
- net NRST: now also J2.2 (Pin_2)
- net SWCLK: now also J2.3 (Pin_3)
- net SWDIO: now also J2.4 (Pin_4)
- net VDD: now also C13.2, C34.1, J2.1 (Pin_1), J5.3 (Pin_3)
- net MISC2: no longer names the net of U17.41 (PB5)
- net ~HBRIDGE_HSIDE renamed ~HALFBRIDGE_HSIDE
- net ~HBRIDGE_LSIDE renamed ~HALFBRIDGE_LSIDE
- new net VCC: C33.1, J5.1 (Pin_1)
- no-connect marks 13 -> 16

Commit message: v1.3 Layout added & schematic update.
Parts:
- removed C32, C33: 100n, Capacitor_SMD:C_0805_2012Metric, symbol Device:C_Small
- removed J2: Conn_01x05, Connector_PinHeader_2.54mm:PinHeader_1x05_P2.54mm_Vertical, symbol Connector_Generic:Conn_01x05
- removed J5: Conn_01x08, Connector_PinHeader_2.54mm:PinHeader_1x08_P2.54mm_Vertical, symbol Connector_Generic:Conn_01x08
- added J2: Conn_01x08, Connector_PinHeader_2.54mm:PinHeader_1x08_P2.54mm_Vertical, symbol Connector_Generic:Conn_01x08
Connections:
- net +5V: now also C13.1, J2.1 (Pin_1)
- net GND: now also C13.2, J2.8 (Pin_8); no longer C13.1
- net MISC0: now also J2.4 (Pin_4)
- net MISC1: now also J2.3 (Pin_3)
- net NRST: now also J2.5 (Pin_5)
- net SWCLK: now also J2.6 (Pin_6)
- net SWDIO: now also J2.7 (Pin_7)
- net VDD: now also J2.2 (Pin_2); no longer C13.2
Other:
- moved on the sheet: C13, C34
