File: v1.3/Hardware/PowerSources.kicad_sch (KiCad schematic)
At the start: 35 parts, among them Q10 BC857C, Q7 BC847C, Q8 BC857C, Q9 BC847C, T3 Transformer_1P_2S, U14 TLV1117-33, U6 L7805, U7 TLV73333PDBV

Commit message: v1.3 Schematic, footprints and BOM updated.
Parts:
- C35: renamed from C?; footprint (none) -> Capacitor_THT:CP_Radial_D10.0mm_P5.00mm
- C47: footprint (none) -> Capacitor_THT:CP_Radial_D13.0mm_P5.00mm
- D10, D11, D12, D13: footprint (none) -> Diode_SMD:D_SMA
- D18, D19, D20, D21: footprint (none) -> Diode_SMD:D_SOD-123
- D6: renamed from D?; footprint (none) -> Diode_SMD:D_SMA
- T1: renamed from T?; footprint (none) -> oe_transformer:ASL151212

Commit message: v1.3 Layout added & schematic update.
Other:
- moved on the sheet: C47, D7
