File: v1.3/Hardware/WaveUltrasonics.kicad_pcb (KiCad board)
At the start: 2 copper layers, 257 x 128 mm, 216 parts, among them J1 MAINS_IN, J10 DG25C-B-04P-13-00AH, J2 L-KLS1-207-2-08-S, J3 Screw_Terminal_01x03, J4 DS1069-02MVW6X, J5 Conn_01x04, J6 DS1069-04MVW6X, J7 DS1069-02MVW6X, J8 DS1069-04MVW6X, J9 DG25C-B-04P-13-00AH, Q1 IXGH48N60C3D1, Q10 BC556, Q17 MMBT3904, Q18 MMBT3904, Q19 MMBT3904, Q2 IXGH48N60C3D1, Q20 MMBT3904, Q21 BC817, Q22 BC817, Q23 BC817, Q24 BC817, Q5 BC546, Q6 BC556, Q7 BC546, Q8 BC556, Q9 BC546, T2 Transformer_1P_2S, T3 Transformer_1P_2S, U1 4N39, U10 ACPL-7900, U12 OPA228, U13 L78L05_SOT89, U14 TLV1117-33, U15 4N25, U16 ADM2483xRW, U17 STM32F334C8Tx, U2 4N39, U3 MCP6024, U4 ACPL-7900, U6 L7805, U7 TLV73333PDBV, U8 HCPL-3120, U9 HCPL-3120, Y1 8MHz

Commit message: v1.3 Layout added & schematic update.
Parts:
- removed C20, C37: 820n 400VDC, Capacitor_THT:C_Rect_L24.0mm_W10.1mm_P22.50mm_MKT
- removed C26, C48, C59, C60, C66, C70, C71: 100n, Capacitor_SMD:C_0805_2012Metric
- removed C32: 6.8n 400VAC, Capacitor_THT:C_Rect_L18.0mm_W5.0mm_P15.00mm_FKS3_FKP3
- removed C33, C72: 15n 300VAC, Capacitor_THT:C_Rect_L18.0mm_W5.0mm_P15.00mm_FKS3_FKP3
- removed C45, C46: 470u 35v, Capacitor_THT:CP_Radial_D10.0mm_P5.00mm
- removed C76: 1000u 35v, Capacitor_THT:CP_Radial_D12.5mm_P5.00mm
- removed D26, D27, D28: D, Diode_SMD:D_MiniMELF
- removed D8, D9: 15v, Diode_THT:D_DO-35_SOD27_P7.62mm_Horizontal
- removed J5: Conn_01x04, Connector_PinHeader_2.54mm:PinHeader_1x04_P2.54mm_Vertical
- removed J9: DG25C-B-04P-13-00AH, oe_connector:DG25C-B-04P-13-00AH
- removed L1: EMIFilter_LL_2314, oe_inductor:EPCOS_B82721A
- removed Q17: MMBT3904, Package_TO_SOT_SMD:SOT-23
- removed Q21, Q22: BC817, Package_TO_SOT_SMD:SOT-23
- removed Q5: BC546, Package_TO_SOT_THT:TO-92_Inline_Wide
- removed Q6: BC556, Package_TO_SOT_THT:TO-92_Inline_Wide
- removed R33, R34: 1k %1, Resistor_SMD:R_0805_2012Metric
- removed R37, R38: 1k, Resistor_THT:R_Axial_DIN0204_L3.6mm_D1.6mm_P5.08mm_Horizontal
- removed R47, R48, R51, R62, R64: 4.7k, Resistor_SMD:R_0805_2012Metric
- removed R49, R50: 1M, Resistor_SMD:R_0805_2012Metric
- removed R53: 120R, Resistor_SMD:R_0805_2012Metric
- removed R63, R65: 2.2k, Resistor_SMD:R_0805_2012Metric
- removed R75: 6.8k 7W, Resistor_THT:R_Axial_Power_L25.0mm_W9.0mm_P30.48mm
- removed T2: Transformer_1P_2S, oe_transformer:ASL151212
- removed TP13, TP14: TestPoint_2Pole, Connector_PinHeader_2.54mm:PinHeader_1x02_P2.54mm_Vertical
- removed U12: OPA228, Package_SO:SOIC-8_3.9x4.9mm_P1.27mm
- removed U16: ADM2483xRW, Package_SO:SOIC-16W_7.5x10.3mm_P1.27mm
- added C22: 22nF 2000VDC, Capacitor_THT:C_Rect_L26.5mm_W10.5mm_P22.50mm_MKS4, F.Cu at (258.6, 152.9)
- added Q3: BC817-40, Package_TO_SOT_SMD:SOT-23, F.Cu at (202.1, 61.5)
- added Q4: MMBT3904, Package_TO_SOT_SMD:SOT-23, F.Cu at (120.8, 168.1)
- added T1: ASL151212, oe_transformer:ASL151212, F.Cu at (104.9, 81.2)
- C10: footprint Capacitor_SMD:C_0805_2012Metric -> Capacitor_SMD:C_1206_3216Metric
- C13: value 1u -> 100n
- C16, C17, C18, C19: value 1u 35v -> 2.2u 50v; footprint Capacitor_THT:CP_Radial_D5.0mm_P2.50mm -> Capacitor_SMD:C_0805_2012Metric
- C23: value 2.2n 400VAC -> 1.5n 400VAC; footprint Capacitor_THT:C_Rect_L13.0mm_W4.0mm_P10.00mm_FKS3_FKP3_MKS4 -> Capacitor_THT:C_Rect_L18.0mm_W5.0mm_P15.00mm_FKS3_FKP3
- C25: value 1.5n 400VAC -> 1.5n 1600VDC
- C27: value 6.8n 400VAC -> 10nF 1600VDC; footprint Capacitor_THT:C_Rect_L18.0mm_W5.0mm_P15.00mm_FKS3_FKP3 -> Capacitor_THT:C_Rect_L18.0mm_W6.0mm_P15.00mm_FKS3_FKP3
- C28, C30: value 6.8n 400VAC -> 22nF 2000VDC; footprint Capacitor_THT:C_Rect_L18.0mm_W5.0mm_P15.00mm_FKS3_FKP3 -> Capacitor_THT:C_Rect_L26.5mm_W10.5mm_P22.50mm_MKS4
- C29, C31: value 15n 300VAC -> 10nF 1600VDC; footprint Capacitor_THT:C_Rect_L18.0mm_W5.0mm_P15.00mm_FKS3_FKP3 -> Capacitor_THT:C_Rect_L18.0mm_W6.0mm_P15.00mm_FKS3_FKP3
- C34: value 6.8n 400VAC -> 100n; footprint Capacitor_THT:C_Rect_L18.0mm_W5.0mm_P15.00mm_FKS3_FKP3 -> Capacitor_SMD:C_0805_2012Metric
- C35: value 15n 300VAC -> 1000u 25v; footprint Capacitor_THT:C_Rect_L18.0mm_W5.0mm_P15.00mm_FKS3_FKP3 -> Capacitor_THT:CP_Radial_D10.0mm_P5.00mm
- C4, C41, C6, C7: value 33n %5 -> 1n %5
- C44: value 470p %5 -> 47n %5; footprint Capacitor_SMD:C_0805_2012Metric -> Capacitor_SMD:C_1206_3216Metric
- C47: value 1000u 35v -> 2200u 25v; footprint Capacitor_THT:CP_Radial_D12.5mm_P5.00mm -> Capacitor_THT:CP_Radial_D13.0mm_P5.00mm
- C73: value 2.2n 400VAC -> 1.5n 1600VDC; footprint Capacitor_THT:C_Rect_L13.0mm_W4.0mm_P10.00mm_FKS3_FKP3_MKS4 -> Capacitor_THT:C_Rect_L18.0mm_W5.0mm_P15.00mm_FKS3_FKP3
- D1, D3: value CLA50E1200HB -> DSEI60-06A; footprint Package_TO_SOT_THT:TO-247-3_Vertical -> Package_TO_SOT_THT:TO-247-2_Vertical
- D10, D11, D12, D13: value D -> M7-KT; footprint Diode_THT:D_DO-35_SOD27_P7.62mm_Horizontal -> Diode_SMD:D_SMA
- D18, D19, D20, D21: footprint Diode_THT:D_DO-35_SOD27_P7.62mm_Horizontal -> Diode_SMD:D_SOD-123
- D5, D6: value 1N4007 -> M7-KT; footprint Diode_THT:D_A-405_P10.16mm_Horizontal -> Diode_SMD:D_SMA
- J1: value MAINS_IN -> DG25C-B-03P-13-00AH
- J2: value L-KLS1-207-2-08-S -> Conn_01x08; footprint Connector_PinHeader_2.54mm:PinHeader_2x04_P2.54mm_Vertical -> Connector_PinHeader_2.54mm:PinHeader_1x08_P2.54mm_Vertical
- J3: value Screw_Terminal_01x03 -> DG25C-B-03P-13-00AH
- J4: value DS1069-02MVW6X -> DG25C-B-03P-13-00AH; footprint Connector_JST:JST_EH_B2B-EH-A_1x02_P2.50mm_Vertical -> oe_connector:DG25C-B-03P-13-00AH
- J6: value DS1069-04MVW6X -> DS1069-02MVW6X; footprint Connector_JST:JST_EH_B4B-EH-A_1x04_P2.50mm_Vertical -> Connector_JST:JST_EH_B2B-EH-A_1x02_P2.50mm_Vertical
- Q10, Q8: value BC556 -> BC857C; footprint Package_TO_SOT_THT:TO-92_Inline_Wide -> Package_TO_SOT_SMD:SOT-23
- Q23, Q24: value BC817 -> MMBT3904
- Q7, Q9: value BC546 -> BC847C; footprint Package_TO_SOT_THT:TO-92_Inline_Wide -> Package_TO_SOT_SMD:SOT-23
- R1: value 1.5k -> 100R 5W; footprint Resistor_THT:R_Axial_DIN0204_L3.6mm_D1.6mm_P7.62mm_Horizontal -> Resistor_THT:R_Axial_Power_L25.0mm_W9.0mm_P30.48mm
- R10: value 1k %1 -> 10k
- R14, R15: value 6.8R -> 8.2R; footprint Resistor_THT:R_Axial_DIN0207_L6.3mm_D2.5mm_P10.16mm_Horizontal -> Resistor_SMD:R_1206_3216Metric
- R19: value 15R 5W -> 22R 5W
- R2: value 1.5k -> 1k; footprint Resistor_THT:R_Axial_DIN0204_L3.6mm_D1.6mm_P7.62mm_Horizontal -> Resistor_SMD:R_0805_2012Metric
- R27: value 10k -> 120R
- R28: value 2.2k -> 4.7k
- R29, R30: value 120R -> 220R
- R3: value 51R 1/2Watt -> 10R %1; footprint Resistor_SMD:R_1210_3225Metric -> Resistor_SMD:R_0805_2012Metric
- R39, R40, R41, R42: footprint Resistor_THT:R_Axial_DIN0204_L3.6mm_D1.6mm_P5.08mm_Horizontal -> Resistor_SMD:R_0805_2012Metric
- R4: value 51R 1/2Watt -> 4.7k; footprint Resistor_SMD:R_1210_3225Metric -> Resistor_SMD:R_0805_2012Metric
- R59: value 220R -> 470R
- R67, R68: value 120R -> 1k
- R69, R70: value 8.2k -> 4.7k
- R71, R72: value 82R -> 120R
- U1: value 4N39 -> ALZN5B12W; footprint Package_DIP:DIP-6_W7.62mm -> oe_relay:ALZN5B12W
- U2: value 4N39 -> ADM485; footprint Package_DIP:DIP-6_W7.62mm -> Package_SO:SOIC-8_3.9x4.9mm_P1.27mm
- moved J4 258.5 mm to (313.4, 164.0), turned to -90 degrees
- moved C35 191.5 mm to (78.2, 118.6), turned to 0 degrees
- moved C34 160.2 mm to (133.5, 124.3)
- moved G*** 96.2 mm to (237.0, 173.2), turned to 0 degrees
- moved R3 83.8 mm to (81.1, 134.5)
- moved R1 79.4 mm to (238.3, 65.9), turned to 0 degrees
- moved D5 78.1 mm to (202.7, 68.5), turned to -90 degrees
- moved C13 75.1 mm to (130.9, 124.3), turned to 90 degrees
- moved U1 74.3 mm to (219.8, 65.9)
- moved R76 73.7 mm to (278.9, 108.5), turned to 90 degrees
- moved R2 71.6 mm to (198.2, 60.8), turned to 180 degrees
- moved C73 68.8 mm to (299.8, 107.8), turned to -90 degrees
- moved U2 66.2 mm to (115.7, 172.0), turned to -90 degrees
- moved R77 60.9 mm to (290.3, 108.5), turned to 90 degrees
- moved C29 56.4 mm to (302.3, 158.6), turned to 180 degrees
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Connections:
- C13 pad 1: GND2 -> +5V
- C13 pad 2: Vdrive -> GND
- C27 pad 2: Net-(C27-Pad2) -> -VDC
- C28 pad 1: Net-(C27-Pad1) -> /GATE1_GND
- C28 pad 2: Net-(C27-Pad2) -> Net-(C22-Pad2)
- C29 pad 1: Net-(C29-Pad1) -> Net-(C27-Pad1)
- C29 pad 2: /GATE1_GND -> -VDC
- C30 pad 1: Net-(C27-Pad1) -> /GATE1_GND
- C30 pad 2: Net-(C27-Pad2) -> Net-(C22-Pad2)
- C31 pad 1: Net-(C29-Pad1) -> Net-(C27-Pad1)
- C31 pad 2: /GATE1_GND -> -VDC
- C34 pad 1: Net-(C27-Pad1) -> VDD
- C34 pad 2: Net-(C27-Pad2) -> GND
- C35 pad 1: Net-(C29-Pad1) -> VEE
- C35 pad 2: /GATE1_GND -> GND1
- C47 pad 1: VEE -> VCC
- C47 pad 2: GND1 -> GND
- C56 pad 2: -VDC -> Earth_Protective
- C65 pad 1: GND -> +5V
- C65 pad 2: VDD -> GND
- D1 pad 1: +VDC -> Net-(D1-Pad1)
- D3 pad 1: +VDC -> Net-(D1-Pad1)
- D5 pad 2: /PHASE+ -> Net-(D5-Pad2)
- D6 pad 1: /PHASE+ -> VEE
- D7 pad 1: VEE -> VCC
- D7 pad 4: GND1 -> GND
- J1 pad 3: -VDC -> Earth_Protective
- J10 pad 1: Net-(C27-Pad2) -> -VDC
- J10 pad 3: -VDC -> Earth_Protective
- J2 pad 3: /Mcu/HMI_SELF_RX -> /Mcu/MISC1
- J2 pad 4: GND -> /Mcu/MISC0
- J2 pad 5: /Mcu/HMI_SELF_TX -> /Mcu/NRST
- J2 pad 6: /Mcu/MISC2 -> /Mcu/SWCLK
- J2 pad 7: /Mcu/MISC0 -> /Mcu/SWDIO
- J2 pad 8: /Mcu/MISC1 -> GND
- J3 pad 3: -VDC -> Earth_Protective
- J4 pad 1: Vdrive -> Net-(C22-Pad2)
- J4 pad 2: GND2 -> Net-(C27-Pad1)
- J6 pad 1: Net-(C66-Pad2) -> Net-(J6-Pad1)
- Q10 pad 1: Net-(C54-Pad2) -> Net-(D21-Pad2)
- Q10 pad 2: Net-(D21-Pad2) -> Net-(C54-Pad2)
- Q7 pad 1: Net-(C51-Pad1) -> Net-(D18-Pad1)
- Q7 pad 2: Net-(D18-Pad1) -> /GATE1_V+
- Q7 pad 3: /GATE1_V+ -> Net-(C51-Pad1)
- Q8 pad 1: Net-(C52-Pad2) -> Net-(D19-Pad2)
- Q8 pad 2: Net-(D19-Pad2) -> Net-(C52-Pad2)
- Q9 pad 1: Net-(C53-Pad1) -> Net-(D20-Pad1)
- Q9 pad 2: Net-(D20-Pad1) -> /GATE2_V+
- Q9 pad 3: /GATE2_V+ -> Net-(C53-Pad1)
- R1 pad 1: Net-(R1-Pad1) -> Net-(D1-Pad1)
- R10 pad 1: Net-(C44-Pad1) -> VDD
- R10 pad 2: /VDIV -> Net-(Q4-Pad1)
- R16 pad 2: -VDC -> Earth_Protective
- R2 pad 1: Net-(R2-Pad1) -> Net-(Q3-Pad1)
- R2 pad 2: +VDC -> /CONTACTOR_DRV
- R24 pad 2: -VDC -> Earth_Protective
- R25 pad 2: -VDC -> Earth_Protective
- R27 pad 1: GND -> Net-(J6-Pad1)
- R27 pad 2: Net-(R27-Pad2) -> Net-(J6-Pad2)
- R29 pad 1: Net-(D29-Pad1) -> +5V
- R29 pad 2: +5V -> Net-(D29-Pad1)
- R3 pad 1: Net-(R3-Pad1) -> Net-(C44-Pad1)
- R3 pad 2: +5V -> /VDIV
- R30 pad 1: GND -> Net-(D29-Pad2)
- R30 pad 2: Net-(D29-Pad2) -> GND
- R39 pad 1: Net-(C51-Pad1) -> Net-(D18-Pad1)
- R39 pad 2: Net-(D18-Pad1) -> Net-(C51-Pad1)
- R4 pad 1: Net-(R4-Pad1) -> /RS485_RX
- R4 pad 2: +5V -> VDD
- R41 pad 1: Net-(C53-Pad1) -> Net-(D20-Pad1)
- R41 pad 2: Net-(D20-Pad1) -> Net-(C53-Pad1)
- R52 pad 2: -VDC -> Earth_Protective
- R67 pad 1: Net-(Q23-Pad1) -> /~HALFBRIDGE_LSIDE
- R67 pad 2: /~HBRIDGE_LSIDE -> Net-(Q23-Pad1)
- R68 pad 1: Net-(Q24-Pad1) -> /~HALFBRIDGE_HSIDE
- R68 pad 2: /~HBRIDGE_HSIDE -> Net-(Q24-Pad1)
- R69 pad 1: Net-(Q23-Pad1) -> /~HALFBRIDGE_LSIDE
- R69 pad 2: +5V -> VDD
- R70 pad 1: Net-(Q24-Pad1) -> /~HALFBRIDGE_HSIDE
- R70 pad 2: +5V -> VDD
- R73 pad 2: -VDC -> Earth_Protective
- R74 pad 2: -VDC -> Earth_Protective
- R76 pad 2: -VDC -> Earth_Protective
- R77 pad 2: -VDC -> Earth_Protective
- TP11 pad 1: -VDC -> Earth_Protective
- TP2 pad 1: -VDC -> Earth_Protective
- TP3 pad 1: -VDC -> Earth_Protective
- TP6 pad 1: Net-(C27-Pad2) -> -VDC
- U1 pad 1: Net-(R3-Pad1) -> Net-(D5-Pad2)
- U1 pad 3: (no net) -> +VDC
- U1 pad 4: Net-(D1-Pad3) -> Net-(D1-Pad1)
- U1 pad 5: LINE -> Net-(D1-Pad1)
- U1 pad 6: Net-(R1-Pad1) -> +VDC
- U15 pad 6: Net-(R27-Pad2) -> (no net)
- U17 pad 17: /CURRENT_PRO_SENS -> (no net)
- U17 pad 18: /ZERO_CROSSING -> (no net)
- U17 pad 19: /ZERO_CROSSING -> (no net)
- U17 pad 29: /~HBRIDGE_HSIDE -> /~HALFBRIDGE_HSIDE
- U17 pad 30: /~HBRIDGE_LSIDE -> /~HALFBRIDGE_LSIDE
- U17 pad 39: /Mcu/MISC0 -> (no net)
- U17 pad 40: /Mcu/MISC1 -> (no net)
- U17 pad 41: /Mcu/MISC2 -> (no net)
- U17 pad 42: /Mcu/HMI_SELF_TX -> /Mcu/MISC0
- U17 pad 43: /Mcu/HMI_SELF_RX -> /Mcu/MISC1
- U17 pad 45: /THRISTOR0_DRV -> /CONTACTOR_DRV
- U17 pad 46: /THRISTOR1_DRV -> (no net)
- U2 pad 1: Net-(R4-Pad1) -> Net-(Q4-Pad2)
- U2 pad 2: Net-(Q22-Pad3) -> /RS485_DE~RE
- U2 pad 3: (no net) -> /RS485_DE~RE
- U2 pad 4: Net-(D3-Pad3) -> /RS485_TX
- U2 pad 5: NEUT -> GND
- U2 pad 6: Net-(R2-Pad1) -> Net-(J6-Pad2)
Routing:
- net -VDC: track 627.2 -> 0.00 mm, vias 26 -> 0
- net /VDIV: track 365.0 -> 0.00 mm, vias 12 -> 0
- net /RSHUNT: track 356.4 -> 0.00 mm, vias 11 -> 0
- net /GATE1_GND: track 181.0 -> 0.00 mm, vias 5 -> 0
- net +VDC: track 169.1 -> 0.00 mm, vias 6 -> 0
- net NEUT: track 162.6 -> 0.00 mm, vias 6 -> 0
- net LINE: track 145.3 -> 0.00 mm, vias 2 -> 0
- net GND: track 128.4 -> 0.00 mm, vias 59 -> 0
- net /GATE2_V-: track 101.2 -> 0.00 mm, vias 1 -> 0
- net /GATE2_V+: track 95.4 -> 0.00 mm, vias 1 -> 0
- net Net-(C29-Pad1): track 81.9 -> 0.00 mm
- net Net-(D1-Pad3): track 81.3 -> 0.00 mm, vias 4 -> 0
- net /THRISTOR1_DRV: track 77.9 -> 0.00 mm, vias 10 -> 0
- net Net-(D3-Pad3): track 77.7 -> 0.00 mm, vias 4 -> 0
- net /GATE1_V-: track 74.0 -> 0.00 mm, vias 1 -> 0
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- removed copper zone on F.Cu, net +5V
- removed copper zone on B.Cu, net +VDC
- removed copper zone on B.Cu, net -VDC
- removed copper zone on F.Cu, net /GATE1_GND
- removed copper zone on F.Cu, net /RSHUNT
- removed copper zone on B.Cu, net GND
- removed copper zone on F.Cu, net GND
- removed copper zone on B.Cu, net GND1
- removed copper zone on B.Cu, net GND2
- removed copper zone on F.Cu, net LINE
- removed copper zone on F.Cu, net NEUT
- removed copper zone on F.Cu, net Net-(C23-Pad2)
- removed copper zone on F.Cu, net Net-(C25-Pad1)
- removed copper zone on F.Cu, net Net-(C27-Pad1)
- removed copper zone on F.Cu, net Net-(C27-Pad2)
- removed copper zone on F.Cu, net Net-(C43-Pad2)
- removed copper zone on F.Cu, net Net-(C73-Pad2)
- removed copper zone on F.Cu, net VDD
- removed copper zone on F.Cu, net VDDA
- removed copper zone on F.Cu, net VEE
- removed copper zone on F.Cu, net Vdrive
Other:
- board size 257 x 128 mm -> 250 x 128 mm
- board text added: "HBO"
- board text added: "IND_A"
- board text added: "IND_B"
- board text added: "Lattice v1.3"
- board text added: "PRIA"
- board text added: "PRIB"
- board text added: "RSNS+"
- board text added: "VDC-"
- board text added: "VDD"
- board text removed: "3V3"
- board text removed: "BRIDGE_OUT"
- board text removed: "FAN+"
- board text removed: "FAN-"
- board text removed: "GNDI"
- board text removed: "HMISRX"
- board text removed: "HMISTX"
- board text removed: "INDCOMP_A"
- board text removed: "INDCOMP_B"
- board text removed: "INDFILT_A"
- board text removed: "INDFILT_B"
- board text removed: "Lattice v1.2"
- board text removed: "MISC2"
- board text removed: "PHASE+"
- board text removed: "PRIMER+"
- board text removed: "PRIMER-"
- board text removed: "Rshu+"
- board text removed: "Rshu-"
- board text removed: "VDDI"
- board text removed: "VDIV-"
- board text removed: "ZCROSS"
