File: v1.3/Hardware/WaveUltrasonics.kicad_sch (KiCad schematic)
At the start: 0 parts

Commit message: v1.3 Schematic, footprints and BOM updated.
Other:
- sheet HBridge renamed HalfBridge
- sheet HalfBridge: file HBridge.kicad_sch -> HalfBridge.kicad_sch
- sheet Mcu ports: added ~HALFBRIDGE_HSIDE, ~HALFBRIDGE_LSIDE; removed ~HBRIDGE_HSIDE, ~HBRIDGE_LSIDE
